Commit message: test_poppy_control changed to poppy_gazebo

File: poppy_gazebo/urdf/poppy_flat_feet.urdf (robot description, URDF)
Before this commit: robot poppy, 28 links, 27 joints
Links:
- link FR07_left: geometry collision mesh filename=package://poppy_gazebo/meshes/flat_foot/FR07_left.STL; visual mesh filename=package://poppy_gazebo/meshes/flat_foot/FR07_left.STL
- link FR07_right: geometry collision mesh filename=package://poppy_gazebo/meshes/flat_foot/FR07_right.STL; visual mesh filename=package://poppy_gazebo/meshes/flat_foot/FR07_right.STL
- link abdomen: geometry collision mesh filename=package://poppy_gazebo/meshes/flat_foot/abdomen.STL; visual mesh filename=package://poppy_gazebo/meshes/flat_foot/abdomen.STL
- link ankle_left: geometry collision mesh filename=package://poppy_gazebo/meshes/flat_foot/ankle_left.STL; visual mesh filename=package://poppy_gazebo/meshes/flat_foot/ankle_left.STL
- link ankle_right: geometry collision mesh filename=package://poppy_gazebo/meshes/flat_foot/ankle_right.STL; visual mesh filename=package://poppy_gazebo/meshes/flat_foot/ankle_right.STL
- link base_link: geometry collision mesh filename=package://poppy_gazebo/meshes/flat_foot/base_link.STL; visual mesh filename=package://poppy_gazebo/meshes/flat_foot/base_link.STL
- link chest: geometry collision mesh filename=package://poppy_gazebo/meshes/flat_foot/chest.STL; visual mesh filename=package://poppy_gazebo/meshes/flat_foot/chest.STL
- link connector_left: geometry collision mesh filename=package://poppy_gazebo/meshes/flat_foot/connector_left.STL; visual mesh filename=package://poppy_gazebo/meshes/flat_foot/connector_left.STL
- link connector_right: geometry collision mesh filename=package://poppy_gazebo/meshes/flat_foot/connector_right.STL; visual mesh filename=package://poppy_gazebo/meshes/flat_foot/connector_right.STL
- link double_rot: geometry collision mesh filename=package://poppy_gazebo/meshes/flat_foot/double_rot.STL; visual mesh filename=package://poppy_gazebo/meshes/flat_foot/double_rot.STL
- link double_rotation: geometry collision mesh filename=package://poppy_gazebo/meshes/flat_foot/double_rotation.STL; visual mesh filename=package://poppy_gazebo/meshes/flat_foot/double_rotation.STL
- link foot_left: geometry collision mesh filename=package://poppy_gazebo/meshes/flat_foot/foot_left.STL; visual mesh filename=package://poppy_gazebo/meshes/flat_foot/foot_left.STL
- link foot_right: geometry collision mesh filename=package://poppy_gazebo/meshes/flat_foot/foot_right.STL; visual mesh filename=package://poppy_gazebo/meshes/flat_foot/foot_right.STL
- link forearm_left: geometry collision mesh filename=package://poppy_gazebo/meshes/flat_foot/forearm_left.STL; visual mesh filename=package://poppy_gazebo/meshes/flat_foot/forearm_left.STL
- link forearm_right: geometry collision mesh filename=package://poppy_gazebo/meshes/flat_foot/forearm_right.STL; visual mesh filename=package://poppy_gazebo/meshes/flat_foot/forearm_right.STL
- link head: geometry collision mesh filename=package://poppy_gazebo/meshes/flat_foot/head.STL; visual mesh filename=package://poppy_gazebo/meshes/flat_foot/head.STL
- link hip_left: geometry collision mesh filename=package://poppy_gazebo/meshes/flat_foot/hip_left.STL; visual mesh filename=package://poppy_gazebo/meshes/flat_foot/hip_left.STL
- link hip_right: geometry collision mesh filename=package://poppy_gazebo/meshes/flat_foot/hip_right.STL; visual mesh filename=package://poppy_gazebo/meshes/flat_foot/hip_right.STL
- link leg_left: geometry collision mesh filename=package://poppy_gazebo/meshes/flat_foot/leg_left.STL; visual mesh filename=package://poppy_gazebo/meshes/flat_foot/leg_left.STL
- link leg_right: geometry collision mesh filename=package://poppy_gazebo/meshes/flat_foot/leg_right.STL; visual mesh filename=package://poppy_gazebo/meshes/flat_foot/leg_right.STL
- link neck: geometry collision mesh filename=package://poppy_gazebo/meshes/flat_foot/neck.STL; visual mesh filename=package://poppy_gazebo/meshes/flat_foot/neck.STL
- link shoulder_left: geometry collision mesh filename=package://poppy_gazebo/meshes/flat_foot/shoulder_left.STL; visual mesh filename=package://poppy_gazebo/meshes/flat_foot/shoulder_left.STL
- link shoulder_right: geometry collision mesh filename=package://poppy_gazebo/meshes/flat_foot/shoulder_right.STL; visual mesh filename=package://poppy_gazebo/meshes/flat_foot/shoulder_right.STL
- link spine: geometry collision mesh filename=package://poppy_gazebo/meshes/flat_foot/spine.STL; visual mesh filename=package://poppy_gazebo/meshes/flat_foot/spine.STL
- link thigh_right: geometry collision mesh filename=package://poppy_gazebo/meshes/flat_foot/thigh_right.STL; visual mesh filename=package://poppy_gazebo/meshes/flat_foot/thigh_right.STL
- link thight_left: geometry collision mesh filename=package://poppy_gazebo/meshes/flat_foot/thight_left.STL; visual mesh filename=package://poppy_gazebo/meshes/flat_foot/thight_left.STL
- link upper_arm_left: geometry collision mesh filename=package://poppy_gazebo/meshes/flat_foot/upper_arm_left.STL; visual mesh filename=package://poppy_gazebo/meshes/flat_foot/upper_arm_left.STL
- link upper_arm_right: geometry collision mesh filename=package://poppy_gazebo/meshes/flat_foot/upper_arm_right.STL; visual mesh filename=package://poppy_gazebo/meshes/flat_foot/upper_arm_right.STL
